File: 386-amp-33x33.kicad_pcb (KiCad board)
At the start: 2 copper layers, 33 x 32.4 mm, 12 parts, among them J1 INPUT, J2 VCC, U1 LM386

Commit message: getting there
Parts:
- C4: footprint Capacitors_ThroughHole:C_Radial_D5_L6_P2.5 -> Capacitors_ThroughHole:C_Disc_D3_P2.5
Other:
- net class Default: clearance 0.6 -> 0.254; trace_width 0.6 -> 0.508
- rule trace_clearance: 0.6 -> 0.254
- rule trace_min: 0.6 -> 0.254
Changed lines of the file:
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@@
   )
   (setup
-    (last_trace_width 0.6)
-    (trace_clearance 0.6)
+    (last_trace_width 0.508)
+    (trace_clearance 0.254)
     (zone_clearance 0.508)
     (zone_45_only no)
-    (trace_min 0.6)
+    (trace_min 0.254)
     (segment_width 0.2)
     (edge_width 0.1)
@@
     (uvia_drill 0.1)
     (uvias_allowed no)
-    (uvia_min_size 0.2)
-    (uvia_min_drill 0.1)
+    (uvia_min_size 0)
+    (uvia_min_drill 0)
     (pcb_text_width 0.3)
     (pcb_text_size 1.5 1.5)
@@
   (net 11 "Net-(RV1-Pad2)")
   (net_class Default "This is the default net class."
-    (clearance 0.6)
-    (trace_width 0.6)
+    (clearance 0.254)
+    (trace_width 0.508)
     (via_dia 0.6)
     (via_drill 0.4)
@@
   )
   (module Capacitors_ThroughHole:C_Radial_D5_L6_P2.5 (layer F.Cu)
-    (at 168.91 129.54 180)
-    (descr "Radial Electrolytic Capacitor Diameter 5mm x Length 6mm, Pitch 2.5mm")
-    (tags "Electrolytic Capacitor")
-    (fp_text reference C4 (at 1.25 -3.8 180) (layer F.SilkS)
-      (effects (font (size 1 1) (thickness 0.15)))
-    )
-    (fp_text value 0u1 (at 1.25 3.8 180) (layer F.Fab)
-      (effects (font (size 1 1) (thickness 0.15)))
-    )
-    (fp_line (start 1.325 -2.499) (end 1.325 2.499) (layer F.SilkS) (width 0.15))
-    (fp_line (start 1.465 -2.491) (end 1.465 2.491) (layer F.SilkS) (width 0.15))
-    (fp_line (start 1.605 -2.475) (end 1.605 -0.095) (layer F.SilkS) (width 0.15))
-    (fp_line (start 1.605 0.095) (end 1.605 2.475) (layer F.SilkS) (width 0.15))
-    (fp_line (start 1.745 -2.451) (end 1.745 -0.49) (layer F.SilkS) (width 0.15))
-    (fp_line (start 1.745 0.49) (end 1.745 2.451) (layer F.SilkS) (width 0.15))
-    (fp_line (start 1.885 -2.418) (end 1.885 -0.657) (layer F.SilkS) (width 0.15))
-    (fp_line (start 1.885 0.657) (end 1.885 2.418) (layer F.SilkS) (width 0.15))
-    (fp_line (start 2.025 -2.377) (end 2.025 -0.764) (layer F.SilkS) (width 0.15))
-    (fp_line (start 2.025 0.764) (end 2.025 2.377) (layer F.SilkS) (width 0.15))
-    (fp_line (start 2.165 -2.327) (end 2.165 -0.835) (layer F.SilkS) (width 0.15))
-    (fp_line (start 2.165 0.835) (end 2.165 2.327) (layer F.SilkS) (width 0.15))
-    (fp_line (start 2.305 -2.266) (end 2.305 -0.879) (layer F.SilkS) (width 0.15))
-    (fp_line (start 2.305 0.879) (end 2.305 2.266) (layer F.SilkS) (width 0.15))
-    (fp_line (start 2.445 -2.196) (end 2.445 -0.898) (layer F.SilkS) (width 0.15))
-    (fp_line (start 2.445 0.898) (end 2.445 2.196) (layer F.SilkS) (width 0.15))
-    (fp_line (start 2.585 -2.114) (end 2.585 -0.896) (layer F.SilkS) (width 0.15))
-    (fp_line (start 2.585 0.896) (end 2.585 2.114) (layer F.SilkS) (width 0.15))
-    (fp_line (start 2.725 -2.019) (end 2.725 -0.871) (layer F.SilkS) (width 0.15))
-    (fp_line (start 2.725 0.871) (end 2.725 2.019) (layer F.SilkS) (width 0.15))
-    (fp_line (start 2.865 -1.908) (end 2.865 -0.823) (layer F.SilkS) (width 0.15))
-    (fp_line (start 2.865 0.823) (end 2.865 1.908) (layer F.SilkS) (width 0.15))
-    (fp_line (start 3.005 -1.78) (end 3.005 -0.745) (layer F.SilkS) (width 0.15))
-    (fp_line (start 3.005 0.745) (end 3.005 1.78) (layer F.SilkS) (width 0.15))
-    (fp_line (start 3.145 -1.631) (end 3.145 -0.628) (layer F.SilkS) (width 0.15))
-    (fp_line (start 3.145 0.628) (end 3.145 1.631) (layer F.SilkS) (width 0.15))
-    (fp_line (start 3.285 -1.452) (end 3.285 -0.44) (layer F.SilkS) (width 0.15))
-    (fp_line (start 3.285 0.44) (end 3.285 1.452) (layer F.SilkS) (width 0.15))
-    (fp_line (start 3.425 -1.233) (end 3.425 1.233) (layer F.SilkS) (width 0.15))
-    (fp_line (start 3.565 -0.944) (end 3.565 0.944) (layer F.SilkS) (width 0.15))
-    (fp_line (start 3.705 -0.472) (end 3.705 0.472) (layer F.SilkS) (width 0.15))
-    (fp_circle (center 2.5 0) (end 2.5 -0.9) (layer F.SilkS) (width 0.15))
-    (fp_circle (center 1.25 0) (end 1.25 -2.5375) (layer F.SilkS) (width 0.15))
-    (fp_circle (center 1.25 0) (end 1.25 -2.8) (layer F.CrtYd) (width 0.05))
-    (pad 1 thru_hole rect (at 0 0 180) (size 1.3 1.3) (drill 0.8) (layers *.Cu *.Mask F.SilkS)
-      (net 6 "Net-(C4-Pad1)"))
-    (pad 2 thru_hole circle (at 2.5 0 180) (size 1.3 1.3) (drill 0.8) (layers *.Cu *.Mask F.SilkS)
-      (net 7 "Net-(C4-Pad2)"))
-    (model Capacitors_ThroughHole.3dshapes/C_Radial_D5_L6_P2.5.wrl
-      (at (xyz 0.0492126 0 0))
-      (scale (xyz 1 1 1))
-      (rotate (xyz 0 0 90))
-    )
-  )
-  (module Capacitors_ThroughHole:C_Radial_D5_L6_P2.5 (layer F.Cu)
     (at 173.99 128.27 270)
     (descr "Radial Electrolytic Capacitor Diameter 5mm x Length 6mm, Pitch 2.5mm")
@@
     )
   )
+  (module Capacitors_ThroughHole:C_Disc_D3_P2.5 (layer F.Cu)
+    (at 168.91 129.54 180)
+    (descr "Capacitor 3mm Disc, Pitch 2.5mm")
+    (tags Capacitor)
+    (fp_text reference C4 (at 1.25 -2.5 180) (layer F.SilkS)
+      (effects (font (size 1 1) (thickness 0.15)))
+    )
+    (fp_text value 0u1 (at 1.25 2.5 180) (layer F.Fab)
+      (effects (font (size 1 1) (thickness 0.15)))
+    )
+    (fp_line (start -0.9 -1.5) (end 3.4 -1.5) (layer F.CrtYd) (width 0.05))
+    (fp_line (start 3.4 -1.5) (end 3.4 1.5) (layer F.CrtYd) (width 0.05))
+    (fp_line (start 3.4 1.5) (end -0.9 1.5) (layer F.CrtYd) (width 0.05))
+    (fp_line (start -0.9 1.5) (end -0.9 -1.5) (layer F.CrtYd) (width 0.05))
+    (fp_line (start -0.25 -1.25) (end 2.75 -1.25) (layer F.SilkS) (width 0.15))
+    (fp_line (start 2.75 1.25) (end -0.25 1.25) (layer F.SilkS) (width 0.15))
+    (pad 1 thru_hole rect (at 0 0 180) (size 1.3 1.3) (drill 0.8) (layers *.Cu *.Mask F.SilkS)
+      (net 6 "Net-(C4-Pad1)"))
+    (pad 2 thru_hole circle (at 2.5 0 180) (size 1.3 1.3) (drill 0.8001) (layers *.Cu *.Mask F.SilkS)
+      (net 7 "Net-(C4-Pad2)"))
+    (model Capacitors_ThroughHole.3dshapes/C_Disc_D3_P2.5.wrl
+      (at (xyz 0.0492126 0 0))
+      (scale (xyz 1 1 1))
+      (rotate (xyz 0 0 0))
+    )
+  )
   (gr_line (start 151.765 134.62) (end 151.765 102.235) (angle 90) (layer Edge.Cuts) (width 0.1))
   (gr_line (start 184.785 134.62) (end 151.765 134.62) (angle 90) (layer Edge.Cuts) (width 0.1))
@@
   (segment (start 163.894762 115.415) (end 163.894762 115.505238) (width 0.6) (layer F.Cu) (net 4))
   (segment (start 163.83 123.19) (end 163.894762 123.125238) (width 0.6) (layer F.Cu) (net 4))
-  (segment (start 179.705 130.81) (end 182.245 130.81) (width 0.6) (layer F.Cu) (net 5) (status 400000))
-  (segment (start 182.88 130.175) (end 182.88 122.555) (width 0.6) (layer F.Cu) (net 5) (status 800000))
+  (segment (start 179.705 130.81) (end 182.245 130.81) (width 0.6) (layer F.Cu) (net 5))
+  (segment (start 182.88 130.175) (end 182.88 122.555) (width 0.6) (layer F.Cu) (net 5))
   (segment (start 182.245 130.81) (end 182.88 130.175) (width 0.6) (layer F.Cu) (net 5))
-  (segment (start 182.88 122.555) (end 182.88 118.11) (width 0.6) (layer F.Cu) (net 5) (status 400000))
-  (segment (start 180.34 115.57) (end 171.669762 115.57) (width 0.6) (layer F.Cu) (net 5) (status 800000))
+  (segment (start 182.88 122.555) (end 182.88 118.11) (width 0.6) (layer F.Cu) (net 5))
+  (segment (start 180.34 115.57) (end 171.669762 115.57) (width 0.6) (layer F.Cu) (net 5))
   (segment (start 182.88 118.11) (end 180.34 115.57) (width 0.6) (layer F.Cu) (net 5))
-  (segment (start 171.669762 115.57) (end 171.514762 115.415) (width 0.6) (layer F.Cu) (net 5) (status C00000))
+  (segment (start 171.669762 115.57) (end 171.514762 115.415) (width 0.6) (layer F.Cu) (net 5))
   (segment (start 176.53 117.475) (end 174.625 115.57) (width 0.6) (layer F.Cu) (net 5))
   (segment (start 177.8 130.81) (end 176.53 129.54) (width 0.6) (layer F.Cu) (net 5))
   (segment (start 176.53 129.54) (end 176.53 117.475) (width 0.6) (layer F.Cu) (net 5))
-  (segment (start 179.705 130.81) (end 177.8 130.81) (width 0.6) (layer F.Cu) (net 5) (status 400000))
-  (segment (start 174.625 115.57) (end 171.669762 115.57) (width 0.6) (layer F.Cu) (net 5) (status 800000))
-  (segment (start 171.669762 115.57) (end 171.514762 115.415) (width 0.6) (layer F.Cu) (net 5) (status C00000))
+  (segment (start 179.705 130.81) (end 177.8 130.81) (width 0.6) (layer F.Cu) (net 5))
+  (segment (start 174.625 115.57) (end 171.669762 115.57) (width 0.6) (layer F.Cu) (net 5))
   (segment (start 171.669762 115.57) (end 171.514762 115.415) (width 0.6) (layer F.Cu) (net 5))
-  (segment (start 173.99 128.27) (end 170.18 128.27) (width 0.6) (layer F.Cu) (net 6))
+  (segment (start 171.669762 115.57) (end 171.514762 115.415) (width 0.6) (layer F.Cu) (net 5))
+  (segment (start 173.99 128.27) (end 170.18 128.27) (width 0.6) (layer F.Cu) (net 6) (status 10))
   (segment (start 170.18 128.27) (end 168.91 129.54) (width 0.6) (layer F.Cu) (net 6))
   (segment (start 171.514762 117.955) (end 171.93 117.955) (width 0.6) (layer F.Cu) (net 6))
   (segment (start 171.93 117.955) (end 173.99 120.015) (width 0.6) (layer F.Cu) (net 6))
-  (segment (start 173.99 120.015) (end 173.99 128.27) (width 0.6) (layer F.Cu) (net 6))
+  (segment (start 173.99 120.015) (end 173.99 128.27) (width 0.6) (layer F.Cu) (net 6) (status 20))
   (segment (start 171.45 123.19) (end 169.545 123.19) (width 0.6) (layer F.Cu) (net 7))
   (segment (start 166.41 126.325) (end 166.41 129.54) (width 0.6) (layer F.Cu) (net 7))
   (segment (start 169.545 123.19) (end 166.41 126.325) (width 0.6) (layer F.Cu) (net 7))
   (segment (start 161.925 129.54) (end 161.925 131.445) (width 0.6) (layer F.Cu) (net 8) (status 10))
-  (segment (start 172.045 132.715) (end 173.99 130.77) (width 0.6) (layer F.Cu) (net 8))
+  (segment (start 172.045 132.715) (end 173.99 130.77) (width 0.6) (layer F.Cu) (net 8) (status 20))
   (segment (start 163.195 132.715) (end 172.045 132.715) (width 0.6) (layer F.Cu) (net 8))
   (segment (start 161.925 131.445) (end 163.195 132.715) (width 0.6) (layer F.Cu) (net 8))
